File: MEC1003F 2024 Assignment 3.kicad_sch (KiCad schematic)
At the start: 19 parts, among them U1 AP331AWRG-7, U2 AP331AWRG-7, U3 LP2950CDTX-3.3/NOPB

Commit message: Rename and Modify from Assignment 2 Rewrite README with new assignment instructions. Add Flop-Flop Circuit Add footprints for all components.
Parts:
- removed U3: LP2950CDTX-3.3/NOPB, symbol Project Symbols:LP2950CDTX-3.3/NOPB
- added C6, C7: 100nF, Capacitor_SMD:C_0603_1608Metric, symbol Project Symbols:CC0603KRX7R9BB104
- added J3: ~, Project Footprints:CROC MEDIUM, symbol Project Symbols:CROC
- added U2: LP2950CDTX-3.3/NOPB, Project Footprints:TO-252 (LP2950-N) MRF, symbol Project Symbols:LP2950CDTX-3.3/NOPB
- added U4, U5: SN74LVC74APWR, Project Footprints:TSSOP-14 (SN74LVC74A) MRF, symbol Project Symbols:SN74LVC74APWR
- renumbered C2 to C1, C1 to C2, C4 to C3, C5 to C4, C3 to C5, R4 to R1, R3 to R2, R2 to R3, R5 to R4, R1 to R5, U2 to U3
Connections:
- net +3V3: now also C6.1, C7.1, U2.3 (VOUT), U4.1 (1~{CLR}), U4.10 (2~{PRE}), U4.13 (2~{CLR}), U4.14 (VCC), U4.4 (1~{PRE}), U5.1 (1~{CLR}), U5.10 (2~{PRE}), U5.13 (2~{CLR}), U5.14 (VCC), U5.4 (1~{PRE})
- net +BATT: now also U2.1 (IN)
- net GND: now also C6.2, C7.2, U2.2 (GND), U4.7 (GND), U5.7 (GND)
- net RELX_OSC_OUT_3V3: now also U4.3 (1CLK)
- new net OSC_DIV16: J3.1, U5.9 (2Q)
- new net OSC_DIV2: U4.11 (2CLK), U4.5 (1Q)
- new net OSC_DIV4: U4.9 (2Q), U5.3 (1CLK)
- new net OSC_DIV8: U5.11 (2CLK), U5.5 (1Q)
- new net ~{OSC_DIV16}: U5.12 (2D), U5.8 (2~{Q})
- new net ~{OSC_DIV2}: U4.2 (1D), U4.6 (1~{Q})
- new net ~{OSC_DIV4}: U4.12 (2D), U4.8 (2~{Q})
- new net ~{OSC_DIV8}: U5.2 (1D), U5.6 (1~{Q})
Other:
- title: MEC1003F 2024 Assignment 2 -> MEC1003F 2024 Assignment 3
- moved on the sheet: C1, C2, C3, C4, C5, J2, R1, R2, R3, R4, R5, R6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
